Commit message: main

File: pick_and_place/urdf/redbox_v2.urdf.xacro (robot description, xacro)
@@ -13,5 +13,5 @@
         <origin xyz="0.0 0.0 0.0" rpy="0.0 0.0 0.0"/>
         <geometry>
-          <box size="0.065 0.065 0.02"/>
+          <box size="0.03 0.03 0.02"/>
         </geometry>
         <material name="red">
@@ -21,5 +21,5 @@
         <origin xyz="0.0 0.0 0.0" rpy="0.0 0.0 0.0"/>
         <geometry>
-          <box size="0.065 0.065 0.02"/>
+          <box size="0.03 0.03 0.02"/>
         </geometry>
       </collision>

Commit message: main

File: pick_and_place/urdf/redbox_v2.urdf.xacro (robot description, xacro)
@@ -13,5 +13,5 @@
         <origin xyz="0.0 0.0 0.0" rpy="0.0 0.0 0.0"/>
         <geometry>
-          <box size="0.03 0.03 0.02"/>
+          <box size="0.035 0.035 0.06"/>
         </geometry>
         <material name="red">
@@ -21,5 +21,5 @@
         <origin xyz="0.0 0.0 0.0" rpy="0.0 0.0 0.0"/>
         <geometry>
-          <box size="0.03 0.03 0.02"/>
+          <box size="0.035 0.035 0.06"/>
         </geometry>
       </collision>
